File: vive-charge-dock.kicad_sch (KiCad schematic)
At the start: 0 parts

Commit message: Copied the pogo files over as a starting point
Parts:
- added P101: ZX80-B-5S, remote_zx80-b-5s_30_:Hirose_ZX80-B-5S_Slot, symbol remote_zx80-b-5s_30_:ZX80-B-5S
- added R101: 0R, remote_rc0402jr-070rp:R_0402_1005Metric, symbol remote_rc0402jr-070rp:Res
- added TP101, TP102: TP_200_SMD, remote_test_point__2.00_mm:TP_200_SMD, symbol remote_test_point__2.00_mm:Test_Point
Connections:
- new net DN: P101.2 (D-), R101.1
- new net DP: P101.3 (D+), R101.2
- new net GND: P101.5 (GND), TP102.1
- new net VCC: P101.1 (VCC), TP101.1
- no-connect marks 0 -> 1
Other:
- title: (none) -> Main
